File: Adafruit-GPS-Logger-Shield-PCB/Adafruit GPS Logger Shield.sch (EAGLE design)
At the start: 27 parts, among them U1 FGPMMOPA6H, U2 MIC5225-3.3, U3 ARDUINOR3-DIMENSION, U4 4050

Commit message: malo o hardwareu
Parts:
- removed C3: 10uF, microbuilder:CAP_CERAMIC0805
- removed U2: MIC5225-3.3, microbuilder:VREG_SOT23-5
Connections:
- net +5V: no longer C3.P$1, U2.EN, U2.IN
- net 3.3V: no longer U2.OUT
- net GND: no longer C3.P$2, U2.GND
Changed lines of the file:
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@@
 <part name="U$1" library="microbuilder" deviceset="FRAME_A4_ADAFRUIT" device=""/>
 <part name="U1" library="microbuilder" deviceset="GPS_FGPMMOPA6H" device="" value="FGPMMOPA6H"/>
-<part name="U2" library="microbuilder" deviceset="VREG_SOT23-5" device="" value="MIC5225-3.3"/>
 <part name="LED1" library="microbuilder" deviceset="LED" device="0805" value="red"/>
 <part name="R1" library="microbuilder" deviceset="RESISTOR" device="0805" value="1K"/>
@@
 <part name="C2" library="microbuilder" deviceset="CAP_CERAMIC" device="0805" value="10uF"/>
 <part name="U$5" library="microbuilder" deviceset="GND" device=""/>
-<part name="U$6" library="microbuilder" deviceset="GND" device=""/>
 <part name="FB1" library="microbuilder" deviceset="FERRITE" device="0805" value="Ferrite"/>
-<part name="C3" library="microbuilder" deviceset="CAP_CERAMIC" device="0805" value="10uF"/>
 <part name="B1" library="microbuilder" deviceset="BATTERY" device="CR1220_SMT" value="CR1220"/>
 <part name="U$14" library="microbuilder" deviceset="GND" device=""/>
@@
 <part name="GND11" library="supply1" deviceset="GND" device=""/>
 <part name="CN2" library="microbuilder" deviceset="MICROSD" device=""/>
-<part name="U$8" library="microbuilder" deviceset="3.3V" device=""/>
 <part name="U$4" library="microbuilder" deviceset="3.3V" device=""/>
 <part name="JP1" library="adafruit" deviceset="PINHD-1X8" device="BIG" value="D0-D7"/>
@@
 <part name="U$11" library="microbuilder" deviceset="3.3V" device=""/>
 <part name="U$12" library="microbuilder" deviceset="3.3V" device=""/>
-<part name="P+2" library="supply1" deviceset="+5V" device=""/>
 <part name="SW1" library="adafruit" deviceset="DPDT" device="-EG1390"/>
 <part name="JP6" library="adafruit" deviceset="PINHD-1X6" device="B"/>
@@
 <instance part="U$1" gate="G$1" x="0" y="0"/>
 <instance part="U1" gate="G$1" x="78.74" y="144.78"/>
-<instance part="U2" gate="G$1" x="33.02" y="99.06"/>
 <instance part="LED1" gate="G$1" x="40.64" y="144.78" rot="R180"/>
 <instance part="R1" gate="G$1" x="30.48" y="144.78"/>
@@
 <instance part="C2" gate="G$1" x="58.42" y="93.98"/>
 <instance part="U$5" gate="G$1" x="58.42" y="88.9"/>
-<instance part="U$6" gate="G$1" x="20.32" y="88.9"/>
 <instance part="FB1" gate="G$1" x="15.24" y="162.56"/>
-<instance part="C3" gate="G$1" x="12.7" y="96.52" rot="MR0"/>
 <instance part="B1" gate="G$1" x="48.26" y="119.38" rot="R180"/>
 <instance part="U$14" gate="G$1" x="58.42" y="114.3"/>
@@
 <instance part="GND11" gate="1" x="175.26" y="81.28"/>
 <instance part="CN2" gate="G$1" x="86.36" y="71.12" rot="MR0"/>
-<instance part="U$8" gate="G$1" x="45.72" y="104.14"/>
 <instance part="U$4" gate="G$1" x="10.16" y="162.56"/>
 <instance part="JP1" gate="G$1" x="215.9" y="58.42" smashed="yes" rot="MR270">
@@
 <instance part="U$11" gate="G$1" x="109.22" y="63.5"/>
 <instance part="U$12" gate="G$1" x="76.2" y="38.1"/>
-<instance part="P+2" gate="1" x="20.32" y="106.68" rot="MR0"/>
 <instance part="SW1" gate="1" x="228.6" y="152.4" rot="R180"/>
 <instance part="SW1" gate="2" x="215.9" y="152.4" rot="R180"/>
@@
 <pinref part="U1" gate="G$1" pin="GND@2"/>
 <pinref part="U1" gate="G$1" pin="GND@1"/>
-</segment>
-<segment>
-<wire x1="22.86" y1="96.52" x2="20.32" y2="96.52" width="0.1524" layer="91"/>
-<wire x1="20.32" y1="96.52" x2="20.32" y2="93.98" width="0.1524" layer="91"/>
-<wire x1="20.32" y1="93.98" x2="20.32" y2="91.44" width="0.1524" layer="91"/>
-<wire x1="12.7" y1="93.98" x2="20.32" y2="93.98" width="0.1524" layer="91"/>
-<junction x="20.32" y="93.98"/>
-<pinref part="U2" gate="G$1" pin="GND"/>
-<pinref part="U$6" gate="G$1" pin="GND"/>
-<pinref part="C3" gate="G$1" pin="P$2"/>
 </segment>
 <segment>
@@
 </segment>
 <segment>
-<pinref part="U2" gate="G$1" pin="OUT"/>
-<pinref part="U$8" gate="G$1" pin="3.3V"/>
-<wire x1="43.18" y1="101.6" x2="43.18" y2="104.14" width="0.1524" layer="91"/>
-<wire x1="43.18" y1="104.14" x2="45.72" y2="104.14" width="0.1524" layer="91"/>
-</segment>
-<segment>
 <pinref part="FB1" gate="G$1" pin="P$1"/>
 <pinref part="U$4" gate="G$1" pin="3.3V"/>
@@
 <pinref part="P+10" gate="1" pin="+5V"/>
 </segment>
-<segment>
-<wire x1="22.86" y1="101.6" x2="20.32" y2="101.6" width="0.1524" layer="91"/>
-<wire x1="20.32" y1="101.6" x2="20.32" y2="104.14" width="0.1524" layer="91"/>
-<wire x1="20.32" y1="101.6" x2="12.7" y2="101.6" width="0.1524" layer="91"/>
-<junction x="20.32" y="101.6"/>
-<pinref part="U2" gate="G$1" pin="IN"/>
-<pinref part="C3" gate="G$1" pin="P$1"/>
-<wire x1="22.86" y1="99.06" x2="20.32" y2="99.06" width="0.1524" layer="91"/>
-<pinref part="U2" gate="G$1" pin="EN"/>
-<wire x1="20.32" y1="101.6" x2="20.32" y2="99.06" width="0.1524" layer="91"/>
-<pinref part="P+2" gate="1" pin="+5V"/>
-</segment>
-</net>
+</net>
